Commit message: urdf

File: Project1/simulation_pkg/simulation/urdf/robot_2_0.urdf (robot description, URDF)
Before this commit: robot robot_2_0, 6 links, 5 joints
Links:
- removed link track_gauge
- added link castor_cylinder; visual cylinder length=0.02 radius=0.02
- added link castor_wheel; visual cylinder length=0.1 radius=0.05
- added link front_axle; visual box size=0.02 0.4 0.02
- link castor_arm: geometry visual box size=0.16 0.02 0.02
Joints:
- removed joint castor_joint
- added joint castor_cylinder_joint: type revolute, parent joint_offset, child castor_cylinder, origin xyz=0 0 0 rpy=-0.01 0 0, axis 0 0 1, limit lower=-1.57 upper=1.57 effort=10 velocity=3
- added joint castor_wheel_joint: type fixed, parent castor_arm, child castor_wheel, origin xyz=0 0.2 0 rpy=0 0 0, axis 0 1 0
- added joint joint_offset_castor: type fixed, parent castor_cylinder, child castor_arm, origin xyz=-0.5 0 0 rpy=0 0 0, axis 0 1 0
- joint attach_to_tf: child track_gauge -> front_axle
