Commit message: version 3 urdf complated and working

File: Project1/simulation_pkg/simulation_description/urdf/robot_2_0_old.xacro (robot description, xacro)
@@ -74,5 +74,5 @@
         <origin xyz="0 0 0" rpy="1.57075 0 0" />
         <geometry>
-          <mesh filename="package://simulation_description/description/wheel.dae" scale="0.001 0.001 0.001"/>
+          <cylinder length="${wheel_thick}" radius="${radius}"/>
         </geometry>
       </visual>
@@ -121,5 +121,5 @@
     <origin rpy="0 0 0" xyz="0 0 ${radius}"/>
   </joint>
-  <joint name="left_wheel_joint" type="continuous">
+  <joint name="left_wheel_joint" type="fixed">
     <axis rpy="0 0 0" xyz="0 1 0"/>
     <parent link="moving_platform"/>
@@ -127,5 +127,5 @@
     <origin rpy="0 0 0" xyz="0 ${front_axle} 0"/>
   </joint>
-  <joint name="right_wheel_joint" type="continuous">
+  <joint name="right_wheel_joint" type="fixed">
     <axis rpy="0 0 0" xyz="0 1 0"/>
     <parent link="moving_platform"/>
@@ -152,5 +152,5 @@
     <origin rpy="0 0 0" xyz="0 ${wheel_thick + .5*thickness} 0"/>
   </joint>
- <joint name="castor_wheel_joint" type="continuous">
+ <joint name="castor_wheel_joint" type="fixed">
     <axis rpy="0 0 0" xyz="0 1 0"/>
     <parent link="castor_arm"/>
